File: MULTICONV/RGBHV_RGBS_CONV.sch (KiCad schematic (older format))
At the start: 39 parts, among them J1 DIGITAL RGB, J10 AUDIO1, J11 RGBHV_2, J12 AUDIO2, J15 RGBS_OUT1, J16 RGBS_OUT2, J17 VIN, J2 VGA DB15, J3 ANALOG RGB DA15, J4 X1, J5 DIGITAL_RGBHV_1, J6 ANALOG RGB, J7 DIGITAL_RGBHV_2, J8 SWITCHER, J9 RGBHV_1, U1 OUT_GND_IN_3.3V, U2 74HC86, U3 OUT_IN_GND_3.3V, U4 IN_OUT_GND_3.3V

Commit message: Rev1.5 リリース候補
Parts:
- removed H2, H3, H4: M4, MountingHole:MountingHole_4.3mm_M4_Pad, symbol Mechanical:MountingHole_Pad
- removed J1: DIGITAL RGB, ryuk_lib:DIN 8 PCB, symbol Connector:DIN-8
- removed J4: X1, ryuk_lib:DIN_6_PCB, symbol Connector:DIN-6
- removed J5: DIGITAL_RGBHV_1, Connector_JST:JST_XH_B8B-XH-A_1x08_P2.50mm_Vertical, symbol Connector_Generic:Conn_01x08
- removed J7: DIGITAL_RGBHV_2, Connector_JST:JST_XH_B8B-XH-A_1x08_P2.50mm_Vertical, symbol Connector_Generic:Conn_01x08
- removed U1: OUT_GND_IN_3.3V, Package_TO_SOT_THT:TO-220-3_Vertical, symbol Regulator_Linear:LM7805_TO220
- removed U3: OUT_IN_GND_3.3V, Package_TO_SOT_THT:TO-220-3_Vertical, symbol Regulator_Linear:HT75xx-1-SOT89
- removed U4: IN_OUT_GND_3.3V, Package_TO_SOT_THT:TO-220-3_Vertical, symbol Regulator_Linear:LM1117-3.3
- added C10, C11, C12, C13: 0.1uF, Capacitor_SMD:C_0603_1608Metric, symbol Device:C
- added C2: 510pF, Capacitor_THT:C_Disc_D5.0mm_W2.5mm_P5.00mm, symbol Device:C
- added C7: 0.1uF, Capacitor_THT:C_Disc_D5.0mm_W2.5mm_P5.00mm, symbol Device:C
- added C8, C9: 10uF, Capacitor_SMD:C_1206_3216Metric, symbol Device:C
- added H10, H11, H12, H13, H14, H2, H3, H4, H9: M4, MountingHole:MountingHole_4.3mm_M4, symbol Mechanical:MountingHole
- added H5, H6, H7, H8: M3, MountingHole:MountingHole_3.2mm_M3, symbol Mechanical:MountingHole
- added J13: SE`PARATE RGBHV OUT, Connector_JST:JST_XH_B8B-XH-A_1x08_P2.50mm_Vertical, symbol Connector_Generic:Conn_01x08
- added R12: 620R, Resistor_THT:R_Axial_DIN0207_L6.3mm_D2.5mm_P10.16mm_Horizontal, symbol Device:R
- added R13: 681KR, Resistor_THT:R_Axial_DIN0207_L6.3mm_D2.5mm_P10.16mm_Horizontal, symbol Device:R
- added R14: 470R, Resistor_THT:R_Axial_DIN0207_L6.3mm_D2.5mm_P10.16mm_Horizontal, symbol Device:R
- added R15: 150R, Resistor_SMD:R_0603_1608Metric, symbol Device:R
- added SW1: HSYNC/CSYNC, ryuk_lib:2MS1T1B4M7QES, symbol Switch:SW_SPDT
- added SW2: STRIPPER, ryuk_lib:2MS1T1B4M7QES, symbol Switch:SW_SPDT
- added SW3: BYPASS HC86, ryuk_lib:2MS1T1B4M7QES, symbol Switch:SW_SPDT
- added U1: 3V3_REG, ryuk_lib:PIN_Unified_LDO, symbol ryuk_lib:PIN_Unified_TP220_LDO
- added U3: EL1883, Package_SO:SOIC-8_3.9x4.9mm_P1.27mm, symbol Video:LM1881
- added U4: NL7SZ57, Package_SO:TSOP-6_1.65x3.05mm_P0.95mm, symbol ryuk_lib:NL7SZ57
- H1: footprint MountingHole:MountingHole_4.3mm_M4_Pad -> MountingHole:MountingHole_4.3mm_M4; symbol Mechanical:MountingHole_Pad -> Mechanical:MountingHole
- R1, R2: footprint Resistor_THT:R_Axial_DIN0207_L6.3mm_D2.5mm_P10.16mm_Horizontal -> Resistor_SMD:R_0603_1608Metric
- R3: value 150R -> 10KR; footprint Resistor_THT:R_Axial_DIN0207_L6.3mm_D2.5mm_P10.16mm_Horizontal -> Resistor_SMD:R_0603_1608Metric
Connections:
- net DIGITAL_B is gone; now on an unnamed net: R3.1
- net DIGITAL_G is gone; now on net HSYNC: R2.1
- net DIGITAL_R is gone; now on an unnamed net: R1.1
- net +3V3: now also R3.2, C12.2, C13.2, C7.2, C9.1, U1.3 (OUT), U3.8 (VCC), U4.5 (VCC); no longer C6.1
- net AUDIO_L: now also J13.6 (Pin_6)
- net AUDIO_R: now also J13.7 (Pin_7)
- net B: now also J13.3 (Pin_3); no longer R3.2
- net CSYNC: now also SW3.2 (B); no longer R10.2, R9.2
- net G: now also J13.2 (Pin_2); no longer R2.2
- net GND: now also C11.2, C12.1, C13.1, C2.2, C7.1, C8.2, C9.2, J13.8 (Pin_8), R13.2, U1.2 (GND), U3.4 (GND), U4.2 (GND); no longer C4.2, H1.1
- net HSYNC: now also R12.1, SW1.2 (B), SW2.1 (A); no longer J3.14 (P14)
- net R: now also J13.1 (Pin_1); no longer R1.2
- net VSYNC: now also J15.6 (Pin_6), J16.6 (Pin_6), R1.2
- net at C3.1, J17.2 (Pin_2): now also C8.1, U1.1 (IN); no longer C4.1
- net at R4.2, R5.2, U2.1 (A1): now also U4.1 (B), U4.3 (A)
- net at R10.1, R9.1, U2.11 (Y4): now also R15.1, U4.4 (Y)
- net at R6.2, R7.2, U2.2 (B1): now also R2.2, U4.6 (C)
- net at J3.9 (P9): now also SW1.1 (A)
- new net: R10.2, R15.2, R9.2, SW3.1 (A)
- new net: J3.14 (P14), SW1.3 (C)
- new net: C11.1, C6.1, R13.1, U3.6 (INT)
- new net: C10.1, C2.1, C4.1, R12.2
- new net: C10.2, C4.2, U3.2 (VIDEO)
- new net: SW2.2 (B), SW3.3 (C)
- new net: R14.2, U3.1 (CSYNC)
- new net: J13.5 (Pin_5), U3.3 (FRAME)
- new net: J13.4 (Pin_4), U3.7 (O/E)
- new net: R14.1, SW2.3 (C)
- no-connect marks 22 -> 17
Other:
- note added: "choose between C1 or C13"
- note added: "choose between C3 or C8"
- note added: "choose between C4 or C10"
- note added: "choose between C5 or C9"
- note added: "choose between C6 or C11"
- note added: "choose between C7 or C12"
- note added: "choose between R1 or R5"
- note added: "choose between R2 or R6"
- note added: "choose between R3 or R8"
- note added: "choose between R9 or R15"
- note added: "choose between U2 or U4"
- note removed: "RGBHV OUT\n1 R\n2 G\n3 B\n4 HSYNC\n5 VSYNC\n6 AUDIO_R\n7 AUDIO_L\n8 GND"
- moved on the sheet: C1, C3, C5, J10, J11, J12, J15, J16, J17, J2, J3, J6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
