File: StackMounter/RGBHV_RGBS_CONV_stack.kicad_pcb (KiCad board)
At the start: 2 copper layers, 18 x 106 mm, 5 parts

Commit message: Rev1.5リリース候補
Parts:
- added H3: M4, MountingHole:MountingHole_4.3mm_M4, F.Cu at (63.0, 102.0)
- added H3: M4, MountingHole:MountingHole_4.3mm_M4, F.Cu at (63.0, 96.0)
- added H3: M4, MountingHole:MountingHole_4.3mm_M4, F.Cu at (63.0, 122.0)
- added H3: M4, MountingHole:MountingHole_4.3mm_M4, F.Cu at (63.0, 61.0)
Other:
- board text added: "RGB MULTI CONVERTER MOUNTER REV 1.5 SEP/2022 C) @antarcticlion Licensed under CERN-OHL-W v2"
- board text removed: "RGB MULTI CONVERTER Under Mounter REV 1.0 SEP/2021 (C) @antarcticlion"
Changed lines of the file:
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@@
   (general
     (thickness 1.6)
-    (drawings 18)
+    (drawings 22)
     (tracks 0)
     (zones 0)
-    (modules 5)
+    (modules 9)
     (nets 1)
   )
@@
   )
   (module MountingHole:MountingHole_4.3mm_M4 (layer F.Cu)
+    (at 63 102)
+    (descr "Mounting Hole 4.3mm, no annular, M4")
+    (tags "mounting hole 4.3mm no annular m4")
+    (attr virtual)
+    (fp_text reference H3 (at 0 -5.3) (layer F.SilkS) hide
+      (effects (font (size 1 1) (thickness 0.15)))
+    )
+    (fp_text value M4 (at 0 5.3) (layer F.Fab)
+      (effects (font (size 1 1) (thickness 0.15)))
+    )
+    (fp_circle (center 0 0) (end 4.55 0) (layer F.CrtYd) (width 0.05))
+    (fp_circle (center 0 0) (end 4.3 0) (layer Cmts.User) (width 0.15))
+    (fp_text user %R (at 0.3 0) (layer F.Fab)
+      (effects (font (size 1 1) (thickness 0.15)))
+    )
+    (pad "" np_thru_hole circle (at 0 0) (size 4.3 4.3) (drill 4.3) (layers *.Cu *.Mask))
+  )
+  (module MountingHole:MountingHole_4.3mm_M4 (layer F.Cu)
+    (at 63 96)
+    (descr "Mounting Hole 4.3mm, no annular, M4")
+    (tags "mounting hole 4.3mm no annular m4")
+    (attr virtual)
+    (fp_text reference H3 (at 0 -5.3) (layer F.SilkS) hide
+      (effects (font (size 1 1) (thickness 0.15)))
+    )
+    (fp_text value M4 (at 0 5.3) (layer F.Fab)
+      (effects (font (size 1 1) (thickness 0.15)))
+    )
+    (fp_circle (center 0 0) (end 4.3 0) (layer Cmts.User) (width 0.15))
+    (fp_circle (center 0 0) (end 4.55 0) (layer F.CrtYd) (width 0.05))
+    (fp_text user %R (at 0.3 0) (layer F.Fab)
+      (effects (font (size 1 1) (thickness 0.15)))
+    )
+    (pad "" np_thru_hole circle (at 0 0) (size 4.3 4.3) (drill 4.3) (layers *.Cu *.Mask))
+  )
+  (module MountingHole:MountingHole_4.3mm_M4 (layer F.Cu)
+    (at 63 122)
+    (descr "Mounting Hole 4.3mm, no annular, M4")
+    (tags "mounting hole 4.3mm no annular m4")
+    (attr virtual)
+    (fp_text reference H3 (at 0 -5.3) (layer F.SilkS) hide
+      (effects (font (size 1 1) (thickness 0.15)))
+    )
+    (fp_text value M4 (at 0 5.3) (layer F.Fab)
+      (effects (font (size 1 1) (thickness 0.15)))
+    )
+    (fp_circle (center 0 0) (end 4.55 0) (layer F.CrtYd) (width 0.05))
+    (fp_circle (center 0 0) (end 4.3 0) (layer Cmts.User) (width 0.15))
+    (fp_text user %R (at 0.3 0) (layer F.Fab)
+      (effects (font (size 1 1) (thickness 0.15)))
+    )
+    (pad "" np_thru_hole circle (at 0 0) (size 4.3 4.3) (drill 4.3) (layers *.Cu *.Mask))
+  )
+  (module MountingHole:MountingHole_4.3mm_M4 (layer F.Cu)
+    (at 63 61)
+    (descr "Mounting Hole 4.3mm, no annular, M4")
+    (tags "mounting hole 4.3mm no annular m4")
+    (attr virtual)
+    (fp_text reference H3 (at 0 -5.3) (layer F.SilkS) hide
+      (effects (font (size 1 1) (thickness 0.15)))
+    )
+    (fp_text value M4 (at 0 5.3) (layer F.Fab)
+      (effects (font (size 1 1) (thickness 0.15)))
+    )
+    (fp_circle (center 0 0) (end 4.55 0) (layer F.CrtYd) (width 0.05))
+    (fp_circle (center 0 0) (end 4.3 0) (layer Cmts.User) (width 0.15))
+    (fp_text user %R (at 0.3 0) (layer F.Fab)
+      (effects (font (size 1 1) (thickness 0.15)))
+    )
+    (pad "" np_thru_hole circle (at 0 0) (size 4.3 4.3) (drill 4.3) (layers *.Cu *.Mask))
+  )
+  (module MountingHole:MountingHole_4.3mm_M4 (layer F.Cu)
     (at 55 61)
     (descr "Mounting Hole 4.3mm, no annular, M4")
@@
       (effects (font (size 1 1) (thickness 0.15)))
     )
-    (fp_circle (center 0 0) (end 4.55 0) (layer F.CrtYd) (width 0.05))
-    (fp_circle (center 0 0) (end 4.3 0) (layer Cmts.User) (width 0.15))
+    (fp_circle (center 0 0) (end 4.3 0) (layer Cmts.User) (width 0.15))
+    (fp_circle (center 0 0) (end 4.55 0) (layer F.CrtYd) (width 0.05))
     (fp_text user %R (at 0.3 0) (layer F.Fab)
       (effects (font (size 1 1) (thickness 0.15)))
@@
       (effects (font (size 1 1) (thickness 0.15)))
     )
-    (fp_circle (center 0 0) (end 4.55 0) (layer F.CrtYd) (width 0.05))
-    (fp_circle (center 0 0) (end 4.3 0) (layer Cmts.User) (width 0.15))
+    (fp_circle (center 0 0) (end 4.3 0) (layer Cmts.User) (width 0.15))
+    (fp_circle (center 0 0) (end 4.55 0) (layer F.CrtYd) (width 0.05))
     (fp_text user %R (at 0.3 0) (layer F.Fab)
       (effects (font (size 1 1) (thickness 0.15)))
@@
       (effects (font (size 1 1) (thickness 0.15)))
     )
-    (fp_circle (center 0 0) (end 4.3 0) (layer Cmts.User) (width 0.15))
-    (fp_circle (center 0 0) (end 4.55 0) (layer F.CrtYd) (width 0.05))
+    (fp_circle (center 0 0) (end 4.55 0) (layer F.CrtYd) (width 0.05))
+    (fp_circle (center 0 0) (end 4.3 0) (layer Cmts.User) (width 0.15))
     (fp_text user %R (at 0.3 0) (layer F.Fab)
       (effects (font (size 1 1) (thickness 0.15)))
@@
       (effects (font (size 1 1) (thickness 0.15)))
     )
+    (fp_circle (center 0 0) (end 3.2 0) (layer Cmts.User) (width 0.15))
     (fp_circle (center 0 0) (end 3.45 0) (layer F.CrtYd) (width 0.05))
-    (fp_circle (center 0 0) (end 3.2 0) (layer Cmts.User) (width 0.15))
     (fp_text user %R (at 0.3 0) (layer F.Fab)
       (effects (font (size 1 1) (thickness 0.15)))
@@
       (effects (font (size 1 1) (thickness 0.15)))
     )
-    (fp_circle (center 0 0) (end 4.55 0) (layer F.CrtYd) (width 0.05))
-    (fp_circle (center 0 0) (end 4.3 0) (layer Cmts.User) (width 0.15))
-    (fp_text user %R (at 0.3 0) (layer F.Fab)
-      (effects (font (size 1 1) (thickness 0.15)))
-    )
-    (pad "" np_thru_hole circle (at 0 0) (size 4.3 4.3) (drill 4.3) (layers *.Cu *.Mask))
+    (fp_circle (center 0 0) (end 4.3 0) (layer Cmts.User) (width 0.15))
+    (fp_circle (center 0 0) (end 4.55 0) (layer F.CrtYd) (width 0.05))
+    (fp_text user %R (at 0.3 0) (layer F.Fab)
+      (effects (font (size 1 1) (thickness 0.15)))
+    )
+    (pad "" np_thru_hole circle (at 0 0) (size 4.3 4.3) (drill 4.3) (layers *.Cu *.Mask))
+  )
+  (dimension 6 (width 0.15) (layer Dwgs.User)
+    (gr_text "6.000 mm" (at 79.3 99 90) (layer Dwgs.User)
+      (effects (font (size 1 1) (thickness 0.15)))
+    )
+    (feature1 (pts (xy 63 96) (xy 78.586421 96)))
+    (feature2 (pts (xy 63 102) (xy 78.586421 102)))
+    (crossbar (pts (xy 78 102) (xy 78 96)))
+    (arrow1a (pts (xy 78 96) (xy 78.586421 97.126504)))
+    (arrow1b (pts (xy 78 96) (xy 77.413579 97.126504)))
+    (arrow2a (pts (xy 78 102) (xy 78.586421 100.873496)))
+    (arrow2b (pts (xy 78 102) (xy 77.413579 100.873496)))
+  )
+  (dimension 35 (width 0.15) (layer Dwgs.User)
+    (gr_text "35.000 mm" (at 89.3 78.5 90) (layer Dwgs.User)
+      (effects (font (size 1 1) (thickness 0.15)))
+    )
+    (feature1 (pts (xy 63 61) (xy 88.586421 61)))
+    (feature2 (pts (xy 63 96) (xy 88.586421 96)))
+    (crossbar (pts (xy 88 96) (xy 88 61)))
+    (arrow1a (pts (xy 88 61) (xy 88.586421 62.126504)))
+    (arrow1b (pts (xy 88 61) (xy 87.413579 62.126504)))
+    (arrow2a (pts (xy 88 96) (xy 88.586421 94.873496)))
+    (arrow2b (pts (xy 88 96) (xy 87.413579 94.873496)))
+  )
+  (dimension 35 (width 0.15) (layer Dwgs.User)
+    (gr_text "35.000 mm" (at 89.3 139.5 90) (layer Dwgs.User)
+      (effects (font (size 1 1) (thickness 0.15)))
+    )
+    (feature1 (pts (xy 63 122) (xy 88.586421 122)))
+    (feature2 (pts (xy 63 157) (xy 88.586421 157)))
+    (crossbar (pts (xy 88 157) (xy 88 122)))
+    (arrow1a (pts (xy 88 122) (xy 88.586421 123.126504)))
+    (arrow1b (pts (xy 88 122) (xy 87.413579 123.126504)))
+    (arrow2a (pts (xy 88 157) (xy 88.586421 155.873496)))
+    (arrow2b (pts (xy 88 157) (xy 87.413579 155.873496)))
+  )
+  (gr_text "@antarcticlion\n" (at 54 85 90) (layer B.Cu)
+    (effects (font (size 5 3) (thickness 0.3)) (justify mirror))
+  )
+  (gr_text "@antarcticlion\n" (at 54 85 90) (layer F.Cu)
+    (effects (font (size 5 3) (thickness 0.3)))
+  )
+  (dimension 6 (width 0.15) (layer Dwgs.User)
+    (gr_text "6.000 mm" (at 79.3 64 90) (layer Dwgs.User)
+      (effects (font (size 1 1) (thickness 0.15)))
+    )
+    (feature1 (pts (xy 63 61) (xy 78.586421 61)))
+    (feature2 (pts (xy 63 67) (xy 78.586421 67)))
+    (crossbar (pts (xy 78 67) (xy 78 61)))
+    (arrow1a (pts (xy 78 61) (xy 78.586421 62.126504)))
+    (arrow1b (pts (xy 78 61) (xy 77.413579 62.126504)))
+    (arrow2a (pts (xy 78 67) (xy 78.586421 65.873496)))
+    (arrow2b (pts (xy 78 67) (xy 77.413579 65.873496)))
   )
   (gr_line (start 68 62) (end 58 62) (layer B.SilkS) (width 0.15))
   (gr_line (start 58 62) (end 58 162) (layer B.SilkS) (width 0.15))
-  (gr_text "@antarcticlion\n" (at 63 133 90) (layer B.Cu)
-    (effects (font (size 5 3) (thickness 0.3)) (justify mirror))
-  )
-  (gr_text "@antarcticlion\n" (at 63 133 90) (layer F.Cu)
-    (effects (font (size 5 3) (thickness 0.3)))
-  )
   (gr_line (start 55 56) (end 63 56) (layer Edge.Cuts) (width 0.15))
   (gr_line (start 55 162) (end 63 162) (layer Edge.Cuts) (width 0.15))
@@
   (gr_line (start 50 61) (end 50 157) (layer Edge.Cuts) (width 0.15))
   (gr_arc (start 55 157) (end 50 157) (angle -90) (layer Edge.Cuts) (width 0.15))
-  (gr_text "RGB MULTI CONVERTER Under Mounter\nREV 1.0 SEP/2021 (C) @antarcticlion\n" (at 54 126 90) (layer B.SilkS)
+  (gr_text "RGB MULTI CONVERTER\nMOUNTER\nREV 1.5 SEP/2022 \nC) @antarcticlion\nLicensed under\nCERN-OHL-W v2" (at 60 136 90) (layer B.SilkS)
     (effects (font (size 1.5 1.5) (thickness 0.3)) (justify mirror))
   )
-  (gr_text "RGB MULTI CONVERTER Under Mounter\nREV 1.0 SEP/2021 (C) @antarcticlion\n" (at 54 126 90) (layer F.SilkS)
+  (gr_text "RGB MULTI CONVERTER\nMOUNTER\nREV 1.5 SEP/2022 \nC) @antarcticlion\nLicensed under\nCERN-OHL-W v2" (at 60 136 90) (layer F.SilkS)
     (effects (font (size 1.5 1.5) (thickness 0.3)))
   )
